File: project/ui.kicad_pcb (KiCad board)
At the start: 2 copper layers, 75 x 220 mm, 105 parts, among them J101 POWER, J102 IDC 2x8, J103 RS485, SW501 RotaryEncoder_Switch, SW601 RotaryEncoder_Switch, SW701 RotaryEncoder_Switch, SW801 RotaryEncoder_Switch, SW901 RotaryEncoder_Switch, U101 LM1117-3.3, U102 MODULE_ESP32-DEVKITC-32U, U103 RS485-UART, U201 MAX7219, U202 3641AS, U203 3641AS, U301 MAX7219, U302 3641AS, U303 3641AS, U401 MAX7219, U402 3641AS, U403 3641AS

Commit message: rs485 connector and minor silkscreen and led values fixes
Parts:
- removed kibuzzard-66DED8D5: G***, kibuzzard-66DED8D5
- added kibuzzard-6736B76D: G***, kibuzzard-6736B76D, F.Cu at (197.5, 180.0)
- J3: renamed from J103; footprint Connector_JST:JST_XH_B3B-XH-A_1x03_P2.50mm_Vertical -> Connector_JST:JST_XH_B4B-XH-A_1x04_P2.50mm_Vertical
- R1: renamed from R101; value 330R -> 10k
- R2: renamed from R102; value 100R -> 4k7
- U2: renamed from U102; value MODULE_ESP32-DEVKITC-32U -> esp32-devkitc-v4
- renumbered C101 to C1, C401 to C10, C501 to C11, C502 to C12, C503 to C13, C601 to C14, C602 to C15, C603 to C16, C701 to C17, C702 to C18, C703 to C19, C102 to C2, C801 to C20, C802 to C21, C803 to C22, C901 to C23, C902 to C24, C903 to C25, C103 to C3, C104 to C4, C106 to C5, C105 to C6, C107 to C7, C201 to C8, C301 to C9, D101 to D1, D102 to D2, D103 to D3, G101 to G1, G102 to G2, H101 to H1, H110 to H10, H111 to H11, H112 to H12, H102 to H2, H103 to H3, H104 to H4, H105 to H5, H106 to H6, H107 to H7, H108 to H8, H109 to H9, J101 to J1, J102 to J2, R302 to R10, R303 to R11, R401 to R12, R402 to R13, R403 to R14, R501 to R15, R502 to R16, R503 to R17, R504 to R18, R601 to R19, R602 to R20, R603 to R21, R604 to R22, R701 to R23, R702 to R24, R703 to R25, R704 to R26, R801 to R27, R802 to R28, R803 to R29, R103 to R3, R804 to R30, R901 to R31, R902 to R32, R903 to R33, R904 to R34, R104 to R4, R105 to R5, R201 to R6, R202 to R7, R203 to R8, R301 to R9, SW501 to SW1, SW601 to SW2, SW701 to SW3, SW801 to SW4, SW901 to SW5, TP101 to TP1, U101 to U1, U401 to U10, U402 to U11, U403 to U12, U103 to U3, U201 to U4, U202 to U5, U203 to U6, U301 to U7, U302 to U8, U303 to U9
Connections:
- J3 pad 1: Net-(J103-Pad1) -> GND
- J3 pad 2: Net-(J103-Pad2) -> Net-(U3-PadA)
- U3 pad A: Net-(J103-Pad1) -> Net-(U3-PadA)
- U3 pad G: Net-(J103-Pad2) -> unconnected-(U3-PadG)
Routing:
- net Net-(J103-Pad1): track 52.8 -> 0.00 mm
- net Net-(U3-PadA): track 0.00 -> 49.5 mm
- net Net-(J103-Pad2): track 37.9 -> 0.00 mm
- net 5V: track 79.7 -> 87.2 mm
- net Net-(U3-PadB): track 40.0 -> 39.2 mm
- net GND: vias 1048 -> 1030
Other:
- board text added: "5V 2A"
- board text added: "5V B- A+ GND"
- board text added: "NOTE: Remove RS485 module to flash esp32 via USB"
- board text removed: "5V"
- board text removed: "B- GND A+"
