File: project/ui.kicad_sch (KiCad schematic)
At the start: 36 parts, among them J101 POWER, J102 IDC 2x8, J103 RS485, U101 LM1117-3.3, U102 esp32-devkitc-v4, U103 RS485-UART

Commit message: rs485 connector and minor silkscreen and led values fixes
Parts:
- J3: renamed from J103; footprint Connector_JST:JST_XH_B3B-XH-A_1x03_P2.50mm_Vertical -> Connector_JST:JST_XH_B4B-XH-A_1x04_P2.50mm_Vertical; symbol Connector_Generic:Conn_01x03 -> Connector_Generic:Conn_01x04
- R1: renamed from R101; value 330R -> 10k
- R2: renamed from R102; value 100R -> 4k7
- renumbered C101 to C1, C102 to C2, C103 to C3, C104 to C4, C106 to C5, C105 to C6, C107 to C7, D101 to D1, D102 to D2, D103 to D3, G101 to G1, G102 to G2, H101 to H1, H110 to H10, H111 to H11, H112 to H12, H102 to H2, H103 to H3, H104 to H4, H105 to H5, H106 to H6, H107 to H7, H108 to H8, H109 to H9, J101 to J1, J102 to J2, R103 to R3, R104 to R4, R105 to R5, TP101 to TP1, U101 to U1, U102 to U2, U103 to U3
Connections:
- net 5V: now also J3.4 (Pin_4)
- net GND: now also J3.1 (Pin_1)
- net at U3.A (A+): now also J3.2 (Pin_2); no longer J3.1 (Pin_1)
- net at U3.G: no longer J3.2 (Pin_2)
- no-connect marks 10 -> 12
Other:
- moved on the sheet: C5
