File: project/ui_encoder.kicad_sch (KiCad schematic)
At the start: 8 parts, among them SW501 RotaryEncoder_Switch

Commit message: rs485 connector and minor silkscreen and led values fixes
Parts:
- renumbered C501 to C11, C502 to C12, C503 to C13, R501 to R15, R502 to R16, R503 to R17, R504 to R18, SW501 to SW1
Changed lines of the file:
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@@
   (title_block
     (title "DZF-6020-UV-power-addon / UI board")
-    (date "2024-09-10")
-    (rev "1.0")
+    (date "2024-11-15")
+    (rev "1.1")
   )
   (junction (at 129.54 106.68) (diameter 0) (color 0 0 0 0)
@@
   (symbol (lib_id "Device:R") (at 133.35 91.44 90) (unit 1)
     (in_bom yes) (on_board yes)
-    (property "Reference" "R502" (id 0) (at 133.35 88.9 90))
+    (property "Reference" "R16" (id 0) (at 133.35 88.9 90))
     (property "Value" "100R" (id 1) (at 133.35 91.44 90))
     (property "Footprint" "Resistor_SMD:R_0805_2012Metric_Pad1.20x1.40mm_HandSolder" (id 2) (at 133.35 93.218 90)
@@
   (symbol (lib_id "Device:R") (at 133.35 111.76 90) (unit 1)
     (in_bom yes) (on_board yes)
-    (property "Reference" "R504" (id 0) (at 133.35 109.22 90))
+    (property "Reference" "R18" (id 0) (at 133.35 109.22 90))
     (property "Value" "1K" (id 1) (at 133.35 111.76 90))
     (property "Footprint" "Resistor_SMD:R_0805_2012Metric_Pad1.20x1.40mm_HandSolder" (id 2) (at 133.35 113.538 90)
@@
   (symbol (lib_id "power:GND") (at 157.48 99.06 0) (unit 1)
     (in_bom yes) (on_board yes) (fields_autoplaced)
-    (property "Reference" "#PWR0501" (id 0) (at 157.48 105.41 0)
+    (property "Reference" "#PWR018" (id 0) (at 157.48 105.41 0)
       (effects (font (size 1.27 1.27)) hide)
     )
@@
   (symbol (lib_id "Device:R") (at 133.35 86.36 90) (unit 1)
     (in_bom yes) (on_board yes)
-    (property "Reference" "R501" (id 0) (at 133.35 83.82 90))
+    (property "Reference" "R15" (id 0) (at 133.35 83.82 90))
     (property "Value" "1K" (id 1) (at 133.35 86.36 90))
     (property "Footprint" "Resistor_SMD:R_0805_2012Metric_Pad1.20x1.40mm_HandSolder" (id 2) (at 133.35 88.138 90)
@@
   (symbol (lib_id "Device:RotaryEncoder_Switch") (at 121.92 99.06 0) (mirror y) (unit 1)
     (in_bom yes) (on_board yes)
-    (property "Reference" "SW501" (id 0) (at 121.92 105.41 0))
+    (property "Reference" "SW1" (id 0) (at 121.92 105.41 0))
     (property "Value" "RotaryEncoder_Switch" (id 1) (at 121.92 106.68 0)
       (effects (font (size 1.27 1.27)) hide)
@@
   (symbol (lib_id "Device:C") (at 156.21 95.25 0) (unit 1)
     (in_bom yes) (on_board yes)
-    (property "Reference" "C503" (id 0) (at 160.02 95.25 0)
+    (property "Reference" "C13" (id 0) (at 160.02 95.25 0)
       (effects (font (size 1.27 1.27)) (justify left))
     )
@@
   (symbol (lib_id "Device:R") (at 133.35 106.68 90) (unit 1)
     (in_bom yes) (on_board yes)
-    (property "Reference" "R503" (id 0) (at 133.35 104.14 90))
+    (property "Reference" "R17" (id 0) (at 133.35 104.14 90))
     (property "Value" "100R" (id 1) (at 133.35 106.68 90))
     (property "Footprint" "Resistor_SMD:R_0805_2012Metric_Pad1.20x1.40mm_HandSolder" (id 2) (at 133.35 108.458 90)
@@
   (symbol (lib_id "Device:C") (at 137.16 102.87 0) (unit 1)
     (in_bom yes) (on_board yes)
-    (property "Reference" "C502" (id 0) (at 140.97 102.87 0)
+    (property "Reference" "C12" (id 0) (at 140.97 102.87 0)
       (effects (font (size 1.27 1.27)) (justify left))
     )
@@
   (symbol (lib_id "Device:C") (at 137.16 95.25 0) (unit 1)
     (in_bom yes) (on_board yes)
-    (property "Reference" "C501" (id 0) (at 140.97 95.25 0)
+    (property "Reference" "C11" (id 0) (at 140.97 95.25 0)
       (effects (font (size 1.27 1.27)) (justify left))
     )
