File: project/pwr.kicad_sch (KiCad schematic)
At the start: 29 parts, among them J101 IDC 2x8, U101 USBLC6-2SC6, U102 USBLC6-2SC6, U103 USBLC6-2SC6, U104 USBLC6-2SC6, U105 TMP102AIDRLR, U106 TMP102AIDRLR

Commit message: finalizing design
Parts:
- added C108: 220u, Capacitor_SMD:CP_Elec_10x10.5, symbol Device:C_Polarized
- added D101: ALR, LED_SMD:LED_0805_2012Metric_Pad1.15x1.40mm_HandSolder, symbol Device:LED
- added D102: VCC, LED_SMD:LED_0805_2012Metric_Pad1.15x1.40mm_HandSolder, symbol Device:LED
- added R108, R109: 100R, Resistor_SMD:R_0805_2012Metric_Pad1.20x1.40mm_HandSolder, symbol Device:R
- added TP101: TP_GND, TestPoint:TestPoint_Loop_D2.60mm_Drill1.6mm_Beaded, symbol Connector:TestPoint_Flag
- C101, C102, C103, C104, C105, C106, C107: lcsc# (none) -> C476766
- U101, U102, U103, U104: lcsc# (none) -> C7519
- U105, U106: lcsc# (none) -> C99269
Connections:
- net 3V3: now also C108.1, D102.2 (A), R108.2
- net ALERT_P: now also D101.1 (K)
- net GND: now also C108.2, R109.1, TP101.1
- new net: D102.1 (K), R109.2
- new net: D101.2 (A), R108.1
Other:
- note added: "I2C addr 0x48"
- note added: "I2C addr 0x49"

Commit message: fixing a lot of stuff in power board
Parts:
- removed H101, H103: MountingHole_Pad, MountingHole:MountingHole_3.2mm_M3_Pad_Via, symbol Mechanical:MountingHole_Pad
- added H105, H106: MountingHole_Pad, MountingHole:MountingHole_3.2mm_M3_Pad_Via, symbol Mechanical:MountingHole_Pad
- R109: value 100R -> 1K
- renumbered H106 to H101, H105 to H103
Connections:
- net GND: no longer H104.1
- no-connect marks 0 -> 3

Commit message: rs485 connector and minor silkscreen and led values fixes
Parts:
- D101: value ALR -> OTP
- R109: value 1K -> 4k7
Changed lines of the file:
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@@
   (title_block
     (title "DZF-6020-UV-power-addon / power board")
-    (date "2024-09-02")
-    (rev "1.0")
+    (date "2024-11-15")
+    (rev "1.2")
   )
   (junction (at 182.88 121.92) (diameter 0) (color 0 0 0 0)
@@
     (in_bom yes) (on_board yes)
     (property "Reference" "R109" (id 0) (at 247.65 154.94 90))
-    (property "Value" "1K" (id 1) (at 247.65 157.48 90))
+    (property "Value" "4k7" (id 1) (at 247.65 157.48 90))
     (property "Footprint" "Resistor_SMD:R_0805_2012Metric_Pad1.20x1.40mm_HandSolder" (id 2) (at 247.65 159.258 90)
       (effects (font (size 1.27 1.27)) hide)
@@
     (in_bom yes) (on_board yes)
     (property "Reference" "D101" (id 0) (at 189.23 119.38 0))
-    (property "Value" "ALR" (id 1) (at 189.23 124.46 0))
+    (property "Value" "OTP" (id 1) (at 189.23 124.46 0))
     (property "Footprint" "LED_SMD:LED_0805_2012Metric_Pad1.15x1.40mm_HandSolder" (id 2) (at 189.23 121.92 0)
       (effects (font (size 1.27 1.27)) hide)
@@
     )
     (path "/54e51e51-8059-4b43-bc90-35d548de0390"
-      (reference "D101") (unit 1) (value "ALR") (footprint "LED_SMD:LED_0805_2012Metric_Pad1.15x1.40mm_HandSolder")
+      (reference "D101") (unit 1) (value "OTP") (footprint "LED_SMD:LED_0805_2012Metric_Pad1.15x1.40mm_HandSolder")
     )
     (path "/4281c847-78df-4c5a-b29a-a1ea1920e237"
@@
     )
     (path "/277e44a1-d2d7-4ed6-8c13-c54b3d0a7975"
-      (reference "R109") (unit 1) (value "1K") (footprint "Resistor_SMD:R_0805_2012Metric_Pad1.20x1.40mm_HandSolder")
+      (reference "R109") (unit 1) (value "4k7") (footprint "Resistor_SMD:R_0805_2012Metric_Pad1.20x1.40mm_HandSolder")
     )
     (path "/6690cda8-0978-4a64-83b9-c387a414df32/87976cd2-f39a-4acd-a502-d54a7c7d11e6"

Commit message: using isolated gate driver
Parts:
- renumbered C101 to C1, C102 to C2, C103 to C3, C104 to C4, C105 to C5, C106 to C6, C107 to C7, C108 to C8, D101 to D1, D102 to D2, G101 to G1, G102 to G2, H101 to H1, H102 to H2, H103 to H3, H104 to H4, H105 to H5, H106 to H6, J101 to J1, R101 to R1, R102 to R2, R103 to R3, R104 to R4, R105 to R5, R106 to R6, R107 to R7, R108 to R8, R109 to R9, TP101 to TP1, U101 to U1, U102 to U2, U103 to U3, U104 to U4, U105 to U5, U106 to U6
